Commit message: Did more things.

File: install/robotiq_hande_description/share/robotiq_hande_description/urdf/cylinder_inertial.xacro (robot description, xacro)
@@ -1 +1,17 @@
-/home/cc/ee106a/fa25/class/ee106a-adc/EECS-C106A-Final-Project/src/robotiq_hande_description/urdf/cylinder_inertial.xacro
+<?xml version="1.0"?>
+<robot xmlns:xacro="http://ros.org/wiki/xacro">
+  <xacro:macro name="__robotiq_hande_cylinder_inertial" params="radius height mass *origin">
+    <inertial>
+      <mass value="${mass}"/>
+      <xacro:insert_block name="origin"/>
+      <inertia
+        ixx="${0.0833333 * mass * (3 * (radius * radius) + height * height)}"
+        ixy="0.0"
+        ixz="0.0"
+        iyy="${0.0833333 * mass * (3 * (radius * radius) + height * height)}"
+        iyz="0.0"
+        izz="${0.5 * mass * (radius * radius)}"
+      />
+    </inertial>
+  </xacro:macro>
+</robot>

File: install/robotiq_hande_description/share/robotiq_hande_description/urdf/robotiq_hande_gripper.ros2_control.xacro (robot description, xacro)
@@ -1 +1,43 @@
-/home/cc/ee106a/fa25/class/ee106a-adc/EECS-C106A-Final-Project/src/robotiq_hande_description/urdf/robotiq_hande_gripper.ros2_control.xacro
+<?xml version="1.0"?>
+<robot xmlns:xacro="http://www.ros.org/wiki/xacro">
+  <xacro:macro
+    name="robotiq_hande_ros2_control"
+    params="name prefix grip_pos_min grip_pos_max tty_port baudrate parity data_bits stop_bit slave_id frequency_hz create_socat_tty socat_ip_address socat_port use_fake_hardware"
+  >
+    <ros2_control name="${name}" type="system">
+      <hardware>
+        <xacro:if value="${use_fake_hardware}">
+          <plugin>mock_components/GenericSystem</plugin>
+        </xacro:if>
+        <xacro:unless value="${use_fake_hardware}">
+          <plugin>robotiq_hande_driver/RobotiqHandeHardwareInterface</plugin>
+          <param name="grip_pos_min">${grip_pos_min}</param>
+          <param name="grip_pos_max">${grip_pos_max}</param>
+          <param name="tty_port">${tty_port}</param>
+          <param name="baudrate">${baudrate}</param>
+          <param name="parity">${parity}</param>
+          <param name="data_bits">${data_bits}</param>
+          <param name="stop_bit">${stop_bit}</param>
+          <param name="slave_id">${slave_id}</param>
+          <param name="frequency_hz">${frequency_hz}</param>
+          <param name="create_socat_tty">${create_socat_tty}</param>
+          <param name="socat_ip_address">${socat_ip_address}</param>
+          <param name="socat_port">${socat_port}</param>
+        </xacro:unless>
+      </hardware>
+      <!-- The right finger joint uses the mimic feature -->
+      <joint name="${prefix}robotiq_hande_left_finger_joint">
+        <command_interface name="position">
+          <param name="min">0</param>
+          <param name="max">0.025</param>
+        </command_interface>
+        <state_interface name="position">
+          <param name="initial_value">0.025</param>
+        </state_interface>
+        <state_interface name="velocity">
+          <param name="initial_value">0</param>
+        </state_interface>
+      </joint>
+    </ros2_control>
+  </xacro:macro>
+</robot>

File: install/robotiq_hande_description/share/robotiq_hande_description/urdf/robotiq_hande_gripper.urdf.xacro (robot description, xacro)
@@ -1 +1,37 @@
-/home/cc/ee106a/fa25/class/ee106a-adc/EECS-C106A-Final-Project/src/robotiq_hande_description/urdf/robotiq_hande_gripper.urdf.xacro
+<?xml version="1.0"?>
+<robot xmlns:xacro="http://ros.org/wiki/xacro" name="robotiq_hande_gripper">
+  <xacro:arg name="parent" default="tool0"/>
+  <xacro:arg name="grip_pos_min" default="0"/>
+  <xacro:arg name="grip_pos_max" default="0.025"/>
+  <xacro:arg name="tty_port" default="/tmp/ttyUR"/>
+  <xacro:arg name="baudrate" default="115200"/>
+  <xacro:arg name="parity" default="N"/>
+  <xacro:arg name="data_bits" default="8"/>
+  <xacro:arg name="stop_bit" default="1"/>
+  <xacro:arg name="slave_id" default="9"/>
+  <xacro:arg name="frequency_hz" default="10"/>
+  <xacro:arg name="create_socat_tty" default="false"/>
+  <xacro:arg name="socat_ip_address" default="192.168.100.10"/>
+  <xacro:arg name="socat_port" default="54321"/>
+  <xacro:arg name="use_fake_hardware" default="true"/>
+  <xacro:include filename="$(find robotiq_hande_description)/urdf/robotiq_hande_gripper.xacro"/>
+  <link name="$(arg parent)"/>
+  <xacro:robotiq_hande_gripper
+    name="robotiq_hande_gripper"
+    prefix=""
+    parent="$(arg parent)"
+    grip_pos_min="$(arg grip_pos_min)"
+    grip_pos_max="$(arg grip_pos_max)"
+    tty_port="$(arg tty_port)"
+    baudrate="$(arg baudrate)"
+    parity="$(arg parity)"
+    data_bits="$(arg data_bits)"
+    stop_bit="$(arg stop_bit)"
+    slave_id="$(arg slave_id)"
+    frequency_hz="$(arg frequency_hz)"
+    create_socat_tty="$(arg create_socat_tty)"
+    socat_ip_address="$(arg socat_ip_address)"
+    socat_port="$(arg socat_port)"
+    use_fake_hardware="$(arg use_fake_hardware)"
+  />
+</robot>

File: install/robotiq_hande_description/share/robotiq_hande_description/urdf/robotiq_hande_gripper.xacro (robot description, xacro)
@@ -1 +1,161 @@
-/home/cc/ee106a/fa25/class/ee106a-adc/EECS-C106A-Final-Project/src/robotiq_hande_description/urdf/robotiq_hande_gripper.xacro
+<?xml version="1.0"?>
+<robot xmlns:xacro="http://ros.org/wiki/xacro">
+  <!--
+    Original URDF file by Cristian C Beltran-Hernandez
+  -->
+  <xacro:include filename="$(find robotiq_hande_description)/urdf/robotiq_hande_gripper.ros2_control.xacro"/>
+  <xacro:include filename="$(find robotiq_hande_description)/urdf/cylinder_inertial.xacro"/>
+  <xacro:macro
+    name="robotiq_hande_gripper"
+    params="name
+            prefix
+            parent
+            grip_pos_min
+            grip_pos_max
+            tty_port
+            baudrate
+            parity
+            data_bits
+            stop_bit
+            slave_id
+            use_fake_hardware
+            frequency_hz:=10
+            create_socat_tty:=false
+            socat_ip_address:=192.168.100.10
+            socat_port:=54321
+            coupler_mass:=0.119
+            xyz:='0 0 0'
+            rpy:='0 0 0'"
+  >
+    <!-- ros2_control parameters  -->
+    <xacro:robotiq_hande_ros2_control
+      name="${name}"
+      prefix="${prefix}"
+      grip_pos_min="${grip_pos_min}"
+      grip_pos_max="${grip_pos_max}"
+      tty_port="${tty_port}"
+      baudrate="${baudrate}"
+      parity="${parity}"
+      data_bits="${data_bits}"
+      stop_bit="${stop_bit}"
+      slave_id="${slave_id}"
+      frequency_hz="${frequency_hz}"
+      create_socat_tty="${create_socat_tty}"
+      socat_ip_address="${socat_ip_address}"
+      socat_port="${socat_port}"
+      use_fake_hardware="${use_fake_hardware}"
+    />
+    <!-- Robotiq Hand-E specs -->
+    <!--  + Height added by the IO coupler: 11.0mm -->
+    <!--  + Height added by the Hand-E: 99.0mm -->
+    <!--  + Coupler mass includes the bolts -->
+    <xacro:arg name="coupler_height" default="0.011"/>
+    <xacro:arg name="coupler_shell_height" default="0.0169"/>
+    <xacro:arg name="coupler_parent_cutoff" default="0.003"/>
+    <xacro:arg name="coupler_hande_cutoff" default="0.0029"/>
+    <xacro:arg name="hande_height" default="0.099"/>
+    <xacro:arg name="hande_radius" default="0.0375"/>
+    <joint name="${prefix}robotiq_hande_coupler_joint" type="fixed">
+      <origin xyz="${xyz}" rpy="${rpy}"/>
+      <parent link="${parent}"/>
+      <child link="${prefix}robotiq_hande_coupler"/>
+    </joint>
+    <link name="${prefix}robotiq_hande_coupler">
+      <visual>
+        <geometry>
+          <mesh filename="package://robotiq_hande_description/meshes/io_coupler.dae"/>
+        </geometry>
+      </visual>
+      <collision>
+        <origin xyz="0 0 ${$(arg coupler_shell_height)/2 - $(arg coupler_parent_cutoff)}" rpy="0 0 0"/>
+        <geometry>
+          <cylinder length="$(arg coupler_shell_height)" radius="${$(arg hande_radius) + 0.001}"/>
+        </geometry>
+      </collision>
+      <xacro:__robotiq_hande_cylinder_inertial radius="$(arg hande_radius)" height="$(arg coupler_shell_height)" mass="${coupler_mass}">
+        <origin xyz="0 0 ${$(arg coupler_shell_height) / 2 - $(arg coupler_parent_cutoff)}" rpy="0 0 0"/>
+      </xacro:__robotiq_hande_cylinder_inertial>
+    </link>
+    <joint name="${prefix}robotiq_hande_base_joint" type="fixed">
+      <origin xyz="0 0 $(arg coupler_height)" rpy="0 0 0"/>
+      <parent link="${prefix}robotiq_hande_coupler"/>
+      <child link="${prefix}robotiq_hande_link"/>
+    </joint>
+    <link name="${prefix}robotiq_hande_link">
+      <visual>
+        <origin xyz="0 0 0" rpy="0 0 0"/>
+        <geometry>
+          <mesh filename="package://robotiq_hande_description/meshes/hande.dae" scale="1.0 1.0 1.0"/>
+        </geometry>
+      </visual>
+      <collision>
+        <origin xyz="0 0 ${($(arg hande_height) + $(arg coupler_hande_cutoff) + 0.005) / 2}" rpy="0 0 0"/>
+        <geometry>
+          <cylinder length="${$(arg hande_height) + $(arg coupler_hande_cutoff) + 0.005}" radius="${$(arg hande_radius) + 0.001}"/>
+        </geometry>
+      </collision>
+      <xacro:__robotiq_hande_cylinder_inertial radius="$(arg hande_radius)" height="$(arg hande_height)" mass="0.86387">
+        <origin xyz="0 0 ${$(arg hande_height) / 2}" rpy="0 0 0"/>
+      </xacro:__robotiq_hande_cylinder_inertial>
+    </link>
+    <joint name="${prefix}robotiq_hande_left_finger_joint" type="prismatic">
+      <origin xyz="0 0 $(arg hande_height)" rpy="0 0 0"/>
+      <parent link="${prefix}robotiq_hande_link"/>
+      <child link="${prefix}robotiq_hande_left_finger"/>
+      <axis xyz="1 0 0"/>
+      <limit effort="130" lower="${grip_pos_min}" upper="${grip_pos_max}" velocity="0.15"/>
+    </joint>
+    <link name="${prefix}robotiq_hande_left_finger">
+      <visual>
+        <origin xyz="0 0 0" rpy="0 0 0"/>
+        <geometry>
+          <mesh filename="package://robotiq_hande_description/meshes/finger.dae" scale="1.0 1.0 1.0"/>
+        </geometry>
+      </visual>
+      <collision>
+        <origin xyz="0 0 0" rpy="0 0 0"/>
+        <geometry>
+          <mesh filename="package://robotiq_hande_description/meshes/finger_collision.dae" scale="1.0 1.0 1.0"/>
+        </geometry>
+      </collision>
+      <inertial>
+        <origin xyz="0 0 0" rpy="0 0 0"/>
+        <mass value="0.03804"/>
+        <inertia ixx="1E-9" ixy="0.0" ixz="0.0" iyy="1E-9" iyz="0.0" izz="1E-9"/>
+      </inertial>
+    </link>
+    <joint name="${prefix}robotiq_hande_right_finger_joint" type="prismatic">
+      <origin xyz="0 0 $(arg hande_height)" rpy="0 0 0"/>
+      <parent link="${prefix}robotiq_hande_link"/>
+      <child link="${prefix}robotiq_hande_right_finger"/>
+      <axis xyz="-1 0 0"/>
+      <limit effort="130" lower="${grip_pos_min}" upper="${grip_pos_max}" velocity="0.15"/>
+      <mimic joint="${prefix}robotiq_hande_left_finger_joint" multiplier="1" offset="0"/>
+    </joint>
+    <link name="${prefix}robotiq_hande_right_finger">
+      <visual>
+        <origin xyz="0 0 0" rpy="0 0 ${pi}"/>
+        <geometry>
+          <mesh filename="package://robotiq_hande_description/meshes/finger.dae" scale="1.0 1.0 1.0"/>
+        </geometry>
+      </visual>
+      <collision>
+        <origin xyz="0 0 0" rpy="0 0 ${pi}"/>
+        <geometry>
+          <mesh filename="package://robotiq_hande_description/meshes/finger_collision.dae" scale="1.0 1.0 1.0"/>
+        </geometry>
+      </collision>
+      <inertial>
+        <origin xyz="0 0 0" rpy="0 0 0"/>
+        <mass value="0.03804"/>
+        <inertia ixx="1E-9" ixy="0.0" ixz="0.0" iyy="1E-9" iyz="0.0" izz="1E-9"/>
+      </inertial>
+    </link>
+    <joint name="${prefix}robotiq_hande_end_joint" type="fixed">
+      <origin xyz="0 0 ${$(arg hande_height) + 0.0465}" rpy="0 0 0"/>
+      <parent link="${prefix}robotiq_hande_link"/>
+      <child link="${prefix}robotiq_hande_end"/>
+    </joint>
+    <link name="${prefix}robotiq_hande_end"/>
+  </xacro:macro>
+</robot>
